Commit message: Fixed pedestrian mesh path.

File: npcs/pedestrian/urdf/pedestrian.urdf (robot description, URDF)
Before this commit: robot pedestrian, 1 links, 0 joints
Links:
- link base_link: geometry collision box size=0.24 0.24 0.6; visual mesh filename=package://competition_2019t2/npcs/pedestrian/meshes/walking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 scale=0.3 0.3 0.3
